Commit message: trying to fix gripper comm bug

File: robotiq_s_model_visualization/cfg/s-model_articulated_macro.xacro (robot description, xacro)
@@ -30,4 +30,5 @@
 			</collision>
 		</link>
+		<link name="${prefix}tool0"/>
         <inertial>
             <origin xyz="0 0 0" rpy="0 0 0"/>
@@ -37,5 +38,4 @@
 		<!-- end of link list -->
 		<!-- joint list -->
-		<!-- WARNING: LIMITS NOT CORRECT -->
 		<joint name="${prefix}palm_finger_1_joint" type="revolute">
 			<parent link="${prefix}palm"/>
@@ -43,7 +43,6 @@
 			<axis xyz="0 1 0"/>
 			<origin xyz="-0.0455 0.0214 0.036" rpy="0 3.1416 -1.57"/>
-			<limit lower="-0.16" upper="0.25" effort="100" velocity="100"/>
+			<limit lower="-0.1784" upper="0.192" effort="100" velocity="100"/>
 		</joint>
-		<!-- WARNING: LIMITS NOT CORRECT -->
 		<joint name="${prefix}palm_finger_2_joint" type="revolute">
 			<parent link="${prefix}palm"/>
@@ -51,5 +50,5 @@
 			<axis xyz="0 1 0"/>
 			<origin xyz="-0.0455 0.0214 -0.036" rpy="0 3.1416 -1.57"/>
-			<limit lower="-0.25" upper="0.16" effort="100" velocity="100"/>
+			<limit lower="-0.192" upper="0.1784" effort="100" velocity="100"/>
 		</joint>
 		<joint name="${prefix}palm_finger_middle_joint" type="fixed">
@@ -59,4 +58,9 @@
 			<origin xyz="0.0455 0.0214 0" rpy="0 0 1.57"/>
 		</joint>
+		<joint name="${prefix}palm_tool0" type="fixed">
+			<parent link="${prefix}palm"/>
+			<child link="${prefix}tool0"/>
+			<origin xyz="0.0 0.0875 0.0" rpy="0 0 1.5707"/>
+		</joint>
 		<!-- end of joint list -->
 	</xacro:macro>

File: robotiq_s_model_visualization/cfg/s-model_finger_articulated_macro.xacro (robot description, xacro)
@@ -19,5 +19,5 @@
 			</visual>
 			<collision>
-				<origin xyz="-0.0455 0.0414 0.036" rpy="0 3.1416 -1.57"/>
+				<origin xyz="0.020 0 0" rpy="0 0 0"/>
 				<geometry>
 					<mesh filename="package://robotiq_s_model_visualization/meshes/s-model_articulated/collision/link_0.STL" />
@@ -103,5 +103,4 @@
 		<!-- end of link list -->
 		<!-- joint list -->
-		<!-- WARNING: LIMITS NOT CORRECT -->
 		<joint name="${prefix}joint_1" type="revolute">
 			<parent link="${prefix}link_0"/>
@@ -109,7 +108,6 @@
 			<axis xyz="0 0 1"/>
 			<origin xyz="0.020 0 0" rpy="0 0 0"/>
-			<limit lower="0" upper="3.1416" effort="100" velocity="100"/>
+			<limit lower="0.0495" upper="1.2218" effort="100" velocity="100"/>
 		</joint>
-		<!-- WARNING: LIMITS NOT CORRECT -->
 		<joint name="${prefix}joint_2" type="revolute">
 			<parent link="${prefix}link_1"/>
@@ -117,7 +115,6 @@
 			<axis xyz="0 0 1"/>
 			<origin xyz="0.050 -.028 0" rpy="0 0 -0.52"/>
-			<limit lower="0" upper="3.1416" effort="100" velocity="100"/>
+			<limit lower="0.0" upper="1.5708" effort="100" velocity="100"/>
 		</joint>
-		<!-- WARNING: LIMITS NOT CORRECT -->
 		<joint name="${prefix}joint_3" type="revolute">
 			<parent link="${prefix}link_2"/>
@@ -125,5 +122,5 @@
 			<axis xyz="0 0 1"/>
 			<origin xyz="0.039 0 0" rpy="0 0 0"/>
-			<limit lower="0" upper="3.1416" effort="100" velocity="100"/>
+			<limit lower="-1.2217" upper="-0.0523" effort="100" velocity="100"/>
 		</joint>
 		<!-- end of joint list -->
